Commit message: File verison Updata

File: motoman_mh12_support/urdf/mh12_robot_v1.urdf (robot description, URDF)
Before this commit: robot motoman_mh12, 8 links, 7 joints
Links:
- link base_link: geometry collision mesh filename=package://motoman_mh12_support/meshes/collision/mh12_base_l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; visual mesh filename=package://motoman_mh12_support/meshes/visual/mh12_base_link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 scale=1.3 1.3 1.3
- link link_1_s: geometry collision mesh filename=package://motoman_mh12_support/meshes/collision/mh12_link_1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; visual mesh filename=package://motoman_mh12_support/meshes/visual/mh12_link_1_s.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 scale=1.3 1.3 1.3
- link link_2_l: geometry collision mesh filename=package://motoman_mh12_support/meshes/collision/mh12_link_2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; visual mesh filename=package://motoman_mh12_support/meshes/visual/mh12_link_2_l.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 scale=1.3 1.3 1.3
- link link_3_u: geometry collision mesh filename=package://motoman_mh12_support/meshes/collision/mh12_link_3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; visual mesh filename=package://motoman_mh12_support/meshes/visual/mh12_link_3_u.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 scale=1.3 1.3 1.3
- link link_4_r: geometry collision mesh filename=package://motoman_mh12_support/meshes/collision/mh12_link_4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; visual mesh filename=package://motoman_mh12_support/meshes/visual/mh12_link_4_r.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 scale=1.3 1.3 1.3
- link link_5_b: geometry collision mesh filename=package://motoman_mh12_support/meshes/collision/mh12_link_5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; visual mesh filename=package://motoman_mh12_support/meshes/visual/mh12_link_5_b.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 scale=1.3 1.3 1.3
- link link_6_t: geometry collision mesh filename=package://motoman_mh12_support/meshes/collision/mh12_link_6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; visual mesh filename=package://motoman_mh12_support/meshes/visual/mh12_link_6_t.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 scale=1.3 1.3 1.3
- link tool0: geometry collision mesh filename=package://motoman_mh12_support/meshes/collision/mh12_link_6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; visual mesh filename=package://motoman_mh12_support/meshes/visual/mh12_link_6_t.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 scale=1.3 1.3 1.3
Joints:
- joint joint_1_s: origin xyz=0 0 0.450 rpy=0 0 0 -> xyz=0 0 2.25 rpy=0 0 0
- joint joint_2_l: origin xyz=0.155 0 0 rpy=0 0 0 -> xyz=0.775 0 0 rpy=0 0 0
- joint joint_3_u: origin xyz=0 0 0.614 rpy=0 0 0 -> xyz=0 0 3.07 rpy=0 0 0
- joint joint_4_r: origin xyz=0.640 0 0.200 rpy=0 0 0 -> xyz=3.2 0 1 rpy=0 0 0
- joint joint_6_t-tool0: origin xyz=0.100 0 0 rpy=3.1415926 -1.570796 0 -> xyz=0.500 0 0 rpy=3.1415926 -1.570796 0

File: motoman_mh12_support/urdf/mh12_robot_v2.urdf (robot description, URDF)
Before this commit: robot motoman_mh12, 8 links, 7 joints
Links:
- link base_link: geometry collision mesh filename=package://motoman_mh12_support/meshes/collision/mh12_base_l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; visual mesh filename=package://motoman_mh12_support/meshes/visual/mh12_base_link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 scale=1.31 1.31 1.31
- link link_1_s: geometry collision mesh filename=package://motoman_mh12_support/meshes/collision/mh12_link_1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; visual mesh filename=package://motoman_mh12_support/meshes/visual/mh12_link_1_s.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 scale=1.31 1.31 1.31
- link link_2_l: geometry collision mesh filename=package://motoman_mh12_support/meshes/collision/mh12_link_2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; visual mesh filename=package://motoman_mh12_support/meshes/visual/mh12_link_2_l.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 scale=1.31 1.31 1.31
- link link_3_u: geometry collision mesh filename=package://motoman_mh12_support/meshes/collision/mh12_link_3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; visual mesh filename=package://motoman_mh12_support/meshes/visual/mh12_link_3_u.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 scale=1.31 1.31 1.31
- link link_4_r: geometry collision mesh filename=package://motoman_mh12_support/meshes/collision/mh12_link_4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; visual mesh filename=package://motoman_mh12_support/meshes/visual/mh12_link_4_r.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 scale=1.31 1.31 1.31
- link link_5_b: geometry collision mesh filename=package://motoman_mh12_support/meshes/collision/mh12_link_5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; visual mesh filename=package://motoman_mh12_support/meshes/visual/mh12_link_5_b.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 scale=1.31 1.31 1.31
- link link_6_t: geometry collision mesh filename=package://motoman_mh12_support/meshes/collision/mh12_link_6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; visual mesh filename=package://motoman_mh12_support/meshes/visual/mh12_link_6_t.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 scale=1.31 1.31 1.31
- link tool0: geometry collision mesh filename=package://motoman_mh12_support/meshes/collision/mh12_link_6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; visual mesh filename=package://motoman_mh12_support/meshes/visual/mh12_link_6_t.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 scale=1.31 1.31 1.31
Joints:
- joint joint_1_s: origin xyz=0 0 0.450 rpy=0 0 0 -> xyz=0 0 0 rpy=0 0 0
